File: kicad/pmod-interface-board.kicad_pcb (KiCad board)
At the start: 4 copper layers, 81.7 x 61 mm, 31 parts, among them J1 PMOD Connector 1, J2 PMOD Connector 2, J4 Gameboy Cart Connector, U1 74HCT541, U2 74HCT541, U3 74HC595, U4 74HC595, U5 74HC595, U6 74HC597

Commit message: src/kicad: fixed incorrectly named OE and PL pins to ~OE and ~PL
Connections:
- net /DATA_IN_PL renamed /~{DATA_IN_PL}
- net /DATA_OUT_OE renamed /~{DATA_OUT_OE}
- net DATA_IN_PL_in renamed ~{DATA_IN_PL}_in
- net DATA_OUT_OE_in renamed ~{DATA_OUT_OE}_in
Changed lines of the file:
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@@
 	(net 9 "~{WR}_in")
 	(net 10 "~{RD}_in")
-	(net 11 "DATA_IN_PL_in")
+	(net 11 "~{DATA_IN_PL}_in")
 	(net 12 "ADDR_SCLK_in")
 	(net 13 "DATA_IN_SCLK_in")
 	(net 14 "DATA_OUT_RCLK_in")
-	(net 15 "/DATA_IN_PL")
+	(net 15 "~{DATA_OUT_OE}_in")
 	(net 16 "DATA_IN_SDATA_out")
 	(net 17 "DATA_IN_RCLK_in")
 	(net 18 "DATA_OUT_SCLK_in")
-	(net 19 "DATA_OUT_OE_in")
+	(net 19 "/~{DATA_OUT_OE}")
 	(net 20 "DATA_OUT_SDATA_in")
 	(net 21 "/A5")
@@
 	(net 56 "/DATA_OUT_SDATA")
 	(net 57 "/DATA_OUT_RCLK")
-	(net 58 "/DATA_OUT_OE")
+	(net 58 "/~{DATA_IN_PL}")
 	(net 59 "/DATA_OUT_SCLK")
 	(net 60 "/DATA_IN_SCLK")
@@
 			(layers "*.Cu" "*.Mask")
 			(remove_unused_layers no)
-			(net 58 "/DATA_OUT_OE")
+			(net 19 "/~{DATA_OUT_OE}")
 			(pinfunction "~{OE}")
 			(pintype "input")
@@
 			(layers "*.Cu" "*.Mask")
 			(remove_unused_layers no)
-			(net 19 "DATA_OUT_OE_in")
+			(net 15 "~{DATA_OUT_OE}_in")
 			(pintype "passive")
 		)
@@
 			(layers "*.Cu" "*.Mask")
 			(remove_unused_layers no)
-			(net 11 "DATA_IN_PL_in")
+			(net 11 "~{DATA_IN_PL}_in")
 			(pinfunction "Pin_8")
 			(pintype "passive")
@@
 			(layers "*.Cu" "*.Mask")
 			(remove_unused_layers no)
-			(net 19 "DATA_OUT_OE_in")
+			(net 15 "~{DATA_OUT_OE}_in")
 			(pinfunction "Pin_12")
 			(pintype "passive")
@@
 			(layers "*.Cu" "*.Mask")
 			(remove_unused_layers no)
-			(net 19 "DATA_OUT_OE_in")
+			(net 15 "~{DATA_OUT_OE}_in")
 			(pinfunction "A1")
 			(pintype "input")
@@
 			(layers "*.Cu" "*.Mask")
 			(remove_unused_layers no)
-			(net 11 "DATA_IN_PL_in")
+			(net 11 "~{DATA_IN_PL}_in")
 			(pinfunction "A4")
 			(pintype "input")
@@
 			(layers "*.Cu" "*.Mask")
 			(remove_unused_layers no)
-			(net 15 "/DATA_IN_PL")
+			(net 58 "/~{DATA_IN_PL}")
 			(pinfunction "Y4")
 			(pintype "tri_state")
@@
 			(layers "*.Cu" "*.Mask")
 			(remove_unused_layers no)
-			(net 58 "/DATA_OUT_OE")
+			(net 19 "/~{DATA_OUT_OE}")
 			(pinfunction "Y1")
 			(pintype "tri_state")
@@
 			(layers "*.Cu" "*.Mask")
 			(remove_unused_layers no)
-			(net 15 "/DATA_IN_PL")
+			(net 58 "/~{DATA_IN_PL}")
 			(pinfunction "~{PL}")
 			(pintype "input")
@@
 			(layers "*.Cu" "*.Mask")
 			(remove_unused_layers no)
-			(net 11 "DATA_IN_PL_in")
+			(net 11 "~{DATA_IN_PL}_in")
 			(pintype "passive")
 		)
@@
 	)
 	(segment
-		(start 156.845 114.935)
-		(end 156.845 109.855)
-		(width 0.25)
-		(layer "B.Cu")
-		(net 15)
-	)
-	(segment
-		(start 137.16 111.76)
-		(end 140.97 115.57)
+		(start 114.3 96.52)
+		(end 115.57 97.79)
 		(width 0.25)
-		(layer "B.Cu")
+		(layer "F.Cu")
 		(net 15)
 	)
 	(segment
-		(start 140.97 115.57)
-		(end 156.21 115.57)
+		(start 127 101.6)
+		(end 123.19 97.79)
 		(width 0.25)
-		(layer "B.Cu")
+		(layer "F.Cu")
 		(net 15)
 	)
 	(segment
-		(start 156.21 115.57)
-		(end 156.845 114.935)
+		(start 127 101.6)
+		(end 129.54 101.6)
 		(width 0.25)
-		(layer "B.Cu")
+		(layer "F.Cu")
 		(net 15)
 	)
 	(segment
-		(start 156.845 109.855)
-		(end 162.56 104.14)
+		(start 115.57 97.79)
+		(end 123.19 97.79)
 		(width 0.25)
-		(layer "B.Cu")
+		(layer "F.Cu")
 		(net 15)
 	)
@@
 	)
 	(segment
-		(start 114.3 96.52)
-		(end 115.57 97.79)
-		(width 0.25)
-		(layer "F.Cu")
-		(net 19)
-	)
-	(segment
-		(start 127 101.6)
-		(end 123.19 97.79)
+		(start 148.59 102.87)
+		(end 149.86 104.14)
 		(width 0.25)
 		(layer "F.Cu")
@@
 	)
 	(segment
-		(start 127 101.6)
-		(end 129.54 101.6)
+		(start 137.16 104.14)
+		(end 138.43 102.87)
 		(width 0.25)
 		(layer "F.Cu")
@@
 	)
 	(segment
-		(start 115.57 97.79)
-		(end 123.19 97.79)
+		(start 138.43 102.87)
+		(end 148.59 102.87)
 		(width 0.25)
 		(layer "F.Cu")
@@
 	)
 	(segment
-		(start 148.59 102.87)
-		(end 149.86 104.14)
+		(start 156.845 114.935)
+		(end 156.845 109.855)
 		(width 0.25)
-		(layer "F.Cu")
+		(layer "B.Cu")
 		(net 58)
 	)
 	(segment
-		(start 137.16 104.14)
-		(end 138.43 102.87)
+		(start 137.16 111.76)
+		(end 140.97 115.57)
 		(width 0.25)
-		(layer "F.Cu")
+		(layer "B.Cu")
 		(net 58)
 	)
 	(segment
-		(start 138.43 102.87)
-		(end 148.59 102.87)
+		(start 140.97 115.57)
+		(end 156.21 115.57)
 		(width 0.25)
-		(layer "F.Cu")
+		(layer "B.Cu")
+		(net 58)
+	)
+	(segment
+		(start 156.21 115.57)
+		(end 156.845 114.935)
+		(width 0.25)
+		(layer "B.Cu")
+		(net 58)
+	)
+	(segment
+		(start 156.845 109.855)
+		(end 162.56 104.14)
+		(width 0.25)
+		(layer "B.Cu")
 		(net 58)
 	)
